Commit message: Update miraculous driver for 20260702 SDK

File: ros2_ws/src/arm_motion_stack/arm_description/urdf/arm.urdf.xacro (robot description, xacro)
@@ -2,4 +2,12 @@
 <robot xmlns:xacro="http://www.ros.org/wiki/xacro" name="ARM">
   <xacro:arg name="hardware_type" default="fake"/>
+  <xacro:arg name="can_interface" default="can0"/>
+  <xacro:arg name="baudrate" default="1000"/>
+  <xacro:arg name="node_ids" default="1,2,3,4,5,6"/>
+  <xacro:arg name="reduction_ratio" default="100.0,100.0,100.0,100.0,100.0,100.0"/>
+  <xacro:arg name="position_min" default="0.0,0.0,0.0,0.0,0.0,0.0"/>
+  <xacro:arg name="position_max" default="0.0,0.0,0.0,0.0,0.0,0.0"/>
+  <xacro:arg name="sync_period_us" default="0"/>
+  <xacro:arg name="read_rate_hz" default="100.0"/>
   <xacro:include filename="materials.xacro"/>
   <!-- Converted from urdf/original/ARM.urdf; link and joint names are preserved. -->
@@ -13,4 +21,14 @@
     <child link="tool0"/>
   </joint>
-  <xacro:arm_ros2_control name="ARMSystem" hardware_type="$(arg hardware_type)"/>
+  <xacro:arm_ros2_control
+    name="ARMSystem"
+    hardware_type="$(arg hardware_type)"
+    can_interface="$(arg can_interface)"
+    baudrate="$(arg baudrate)"
+    node_ids="$(arg node_ids)"
+    reduction_ratio="$(arg reduction_ratio)"
+    position_min="$(arg position_min)"
+    position_max="$(arg position_max)"
+    sync_period_us="$(arg sync_period_us)"
+    read_rate_hz="$(arg read_rate_hz)"/>
 </robot>

File: ros2_ws/src/arm_motion_stack/arm_description/urdf/ros2_control.xacro (robot description, xacro)
@@ -1,5 +1,5 @@
 <?xml version="1.0"?>
 <robot xmlns:xacro="http://www.ros.org/wiki/xacro">
-  <xacro:macro name="arm_ros2_control" params="name hardware_type">
+  <xacro:macro name="arm_ros2_control" params="name hardware_type can_interface baudrate node_ids reduction_ratio position_min position_max sync_period_us read_rate_hz">
     <ros2_control name="${name}" type="system">
       <hardware>
@@ -21,11 +21,12 @@
         <xacro:if value="${hardware_type == 'real'}">
           <plugin>miraculous_driver/MiraculousSystem</plugin>
-          <param name="can_interface">can0</param>
-          <param name="baudrate">1000</param>
-          <param name="node_ids">1,2,3,4,5,6</param>
-          <!-- pulses_per_radian = counts_per_rev * gear_ratio / (2*pi). TODO: replace with real per-joint values. -->
-          <param name="pulses_per_radian">1000.0,1000.0,1000.0,1000.0,1000.0,1000.0</param>
-          <param name="sync_period_us">0</param>
-          <param name="read_rate_hz">100.0</param>
+          <param name="can_interface">${can_interface}</param>
+          <param name="baudrate">${baudrate}</param>
+          <param name="node_ids">${node_ids}</param>
+          <param name="reduction_ratio">${reduction_ratio}</param>
+          <param name="position_min">${position_min}</param>
+          <param name="position_max">${position_max}</param>
+          <param name="sync_period_us">${sync_period_us}</param>
+          <param name="read_rate_hz">${read_rate_hz}</param>
         </xacro:if>
       </hardware>

Commit message: Support partial miraculous arm bringup

File: ros2_ws/src/arm_motion_stack/arm_description/urdf/arm.urdf.xacro (robot description, xacro)
@@ -5,5 +5,5 @@
   <xacro:arg name="baudrate" default="1000"/>
   <xacro:arg name="node_ids" default="1,2,3,4,5,6"/>
-  <xacro:arg name="reduction_ratio" default="100.0,100.0,100.0,100.0,100.0,100.0"/>
+  <xacro:arg name="joint_indices" default="0,1,2,3,4,5"/>
   <xacro:arg name="position_min" default="0.0,0.0,0.0,0.0,0.0,0.0"/>
   <xacro:arg name="position_max" default="0.0,0.0,0.0,0.0,0.0,0.0"/>
@@ -27,5 +27,5 @@
     baudrate="$(arg baudrate)"
     node_ids="$(arg node_ids)"
-    reduction_ratio="$(arg reduction_ratio)"
+    joint_indices="$(arg joint_indices)"
     position_min="$(arg position_min)"
     position_max="$(arg position_max)"

File: ros2_ws/src/arm_motion_stack/arm_description/urdf/ros2_control.xacro (robot description, xacro)
@@ -1,5 +1,5 @@
 <?xml version="1.0"?>
 <robot xmlns:xacro="http://www.ros.org/wiki/xacro">
-  <xacro:macro name="arm_ros2_control" params="name hardware_type can_interface baudrate node_ids reduction_ratio position_min position_max sync_period_us read_rate_hz">
+  <xacro:macro name="arm_ros2_control" params="name hardware_type can_interface baudrate node_ids joint_indices position_min position_max sync_period_us read_rate_hz">
     <ros2_control name="${name}" type="system">
       <hardware>
@@ -24,5 +24,5 @@
           <param name="baudrate">${baudrate}</param>
           <param name="node_ids">${node_ids}</param>
-          <param name="reduction_ratio">${reduction_ratio}</param>
+          <param name="joint_indices">${joint_indices}</param>
           <param name="position_min">${position_min}</param>
           <param name="position_max">${position_max}</param>

Commit message: Stabilize miraculous CSP tracking bringup

File: ros2_ws/src/arm_motion_stack/arm_description/urdf/arm.urdf.xacro (robot description, xacro)
@@ -10,4 +10,5 @@
   <xacro:arg name="sync_period_us" default="0"/>
   <xacro:arg name="read_rate_hz" default="100.0"/>
+  <xacro:arg name="state_poll_rate_hz" default="0.0"/>
   <xacro:include filename="materials.xacro"/>
   <!-- Converted from urdf/original/ARM.urdf; link and joint names are preserved. -->
@@ -31,4 +32,5 @@
     position_max="$(arg position_max)"
     sync_period_us="$(arg sync_period_us)"
-    read_rate_hz="$(arg read_rate_hz)"/>
+    read_rate_hz="$(arg read_rate_hz)"
+    state_poll_rate_hz="$(arg state_poll_rate_hz)"/>
 </robot>

File: ros2_ws/src/arm_motion_stack/arm_description/urdf/ros2_control.xacro (robot description, xacro)
@@ -1,5 +1,5 @@
 <?xml version="1.0"?>
 <robot xmlns:xacro="http://www.ros.org/wiki/xacro">
-  <xacro:macro name="arm_ros2_control" params="name hardware_type can_interface baudrate node_ids joint_indices position_min position_max sync_period_us read_rate_hz">
+  <xacro:macro name="arm_ros2_control" params="name hardware_type can_interface baudrate node_ids joint_indices position_min position_max sync_period_us read_rate_hz state_poll_rate_hz">
     <ros2_control name="${name}" type="system">
       <hardware>
@@ -29,4 +29,5 @@
           <param name="sync_period_us">${sync_period_us}</param>
           <param name="read_rate_hz">${read_rate_hz}</param>
+          <param name="state_poll_rate_hz">${state_poll_rate_hz}</param>
         </xacro:if>
       </hardware>

Commit message: Integrate fail-closed MoveIt hardware path

File: ros2_ws/src/arm_motion_stack/arm_description/urdf/arm.urdf.xacro (robot description, xacro)
@@ -4,4 +4,6 @@
   <xacro:arg name="can_interface" default="can0"/>
   <xacro:arg name="baudrate" default="1000"/>
+  <xacro:arg name="encoder_bw" default="19"/>
+  <xacro:arg name="reduction_ratio" default="100.0"/>
   <xacro:arg name="node_ids" default="1,2,3,4,5,6"/>
   <xacro:arg name="joint_indices" default="0,1,2,3,4,5"/>
@@ -11,4 +13,9 @@
   <xacro:arg name="read_rate_hz" default="100.0"/>
   <xacro:arg name="state_poll_rate_hz" default="0.0"/>
+  <xacro:arg name="manual_feedback_timeout_ms" default="5"/>
+  <xacro:arg name="feedback_stale_timeout_ms" default="30"/>
+  <xacro:arg name="enable_emcy_monitor" default="true"/>
+  <xacro:arg name="require_full_arm" default="false"/>
+  <xacro:arg name="require_position_limits" default="false"/>
   <xacro:include filename="materials.xacro"/>
   <!-- Converted from urdf/original/ARM.urdf; link and joint names are preserved. -->
@@ -27,4 +34,6 @@
     can_interface="$(arg can_interface)"
     baudrate="$(arg baudrate)"
+    encoder_bw="$(arg encoder_bw)"
+    reduction_ratio="$(arg reduction_ratio)"
     node_ids="$(arg node_ids)"
     joint_indices="$(arg joint_indices)"
@@ -33,4 +42,9 @@
     sync_period_us="$(arg sync_period_us)"
     read_rate_hz="$(arg read_rate_hz)"
-    state_poll_rate_hz="$(arg state_poll_rate_hz)"/>
+    state_poll_rate_hz="$(arg state_poll_rate_hz)"
+    manual_feedback_timeout_ms="$(arg manual_feedback_timeout_ms)"
+    feedback_stale_timeout_ms="$(arg feedback_stale_timeout_ms)"
+    enable_emcy_monitor="$(arg enable_emcy_monitor)"
+    require_full_arm="$(arg require_full_arm)"
+    require_position_limits="$(arg require_position_limits)"/>
 </robot>

File: ros2_ws/src/arm_motion_stack/arm_description/urdf/ros2_control.xacro (robot description, xacro)
@@ -1,5 +1,5 @@
 <?xml version="1.0"?>
 <robot xmlns:xacro="http://www.ros.org/wiki/xacro">
-  <xacro:macro name="arm_ros2_control" params="name hardware_type can_interface baudrate node_ids joint_indices position_min position_max sync_period_us read_rate_hz state_poll_rate_hz">
+  <xacro:macro name="arm_ros2_control" params="name hardware_type can_interface baudrate encoder_bw reduction_ratio node_ids joint_indices position_min position_max sync_period_us read_rate_hz state_poll_rate_hz manual_feedback_timeout_ms feedback_stale_timeout_ms enable_emcy_monitor require_full_arm require_position_limits">
     <ros2_control name="${name}" type="system">
       <hardware>
@@ -23,4 +23,6 @@
           <param name="can_interface">${can_interface}</param>
           <param name="baudrate">${baudrate}</param>
+          <param name="encoder_bw">${encoder_bw}</param>
+          <param name="reduction_ratio">${reduction_ratio}</param>
           <param name="node_ids">${node_ids}</param>
           <param name="joint_indices">${joint_indices}</param>
@@ -30,4 +32,9 @@
           <param name="read_rate_hz">${read_rate_hz}</param>
           <param name="state_poll_rate_hz">${state_poll_rate_hz}</param>
+          <param name="manual_feedback_timeout_ms">${manual_feedback_timeout_ms}</param>
+          <param name="feedback_stale_timeout_ms">${feedback_stale_timeout_ms}</param>
+          <param name="enable_emcy_monitor">${enable_emcy_monitor}</param>
+          <param name="require_full_arm">${require_full_arm}</param>
+          <param name="require_position_limits">${require_position_limits}</param>
         </xacro:if>
       </hardware>

Commit message: Harden real-arm control and MoveIt safety

File: ros2_ws/src/arm_motion_stack/arm_description/urdf/arm.urdf.xacro (robot description, xacro)
@@ -2,6 +2,6 @@
 <robot xmlns:xacro="http://www.ros.org/wiki/xacro" name="ARM">
   <xacro:arg name="hardware_type" default="fake"/>
-  <xacro:arg name="can_interface" default="can0"/>
-  <xacro:arg name="baudrate" default="1000"/>
+  <xacro:arg name="can_interface" default="can1"/>
+  <xacro:arg name="baudrate" default="0"/>
   <xacro:arg name="encoder_bw" default="19"/>
   <xacro:arg name="reduction_ratio" default="100.0"/>
@@ -11,9 +11,12 @@
   <xacro:arg name="position_max" default="0.0,0.0,0.0,0.0,0.0,0.0"/>
   <xacro:arg name="sync_period_us" default="0"/>
-  <xacro:arg name="read_rate_hz" default="100.0"/>
+  <xacro:arg name="read_rate_hz" default="50.0"/>
   <xacro:arg name="state_poll_rate_hz" default="0.0"/>
-  <xacro:arg name="manual_feedback_timeout_ms" default="5"/>
+  <xacro:arg name="manual_feedback_timeout_ms" default="15"/>
   <xacro:arg name="feedback_stale_timeout_ms" default="30"/>
   <xacro:arg name="enable_emcy_monitor" default="true"/>
+  <xacro:arg name="max_command_step_rad" default="0.005"/>
+  <xacro:arg name="max_following_error_rad" default="0.05"/>
+  <xacro:arg name="following_error_cycles" default="3"/>
   <xacro:arg name="require_full_arm" default="false"/>
   <xacro:arg name="require_position_limits" default="false"/>
@@ -46,4 +49,7 @@
     feedback_stale_timeout_ms="$(arg feedback_stale_timeout_ms)"
     enable_emcy_monitor="$(arg enable_emcy_monitor)"
+    max_command_step_rad="$(arg max_command_step_rad)"
+    max_following_error_rad="$(arg max_following_error_rad)"
+    following_error_cycles="$(arg following_error_cycles)"
     require_full_arm="$(arg require_full_arm)"
     require_position_limits="$(arg require_position_limits)"/>

File: ros2_ws/src/arm_motion_stack/arm_description/urdf/ros2_control.xacro (robot description, xacro)
@@ -1,5 +1,5 @@
 <?xml version="1.0"?>
 <robot xmlns:xacro="http://www.ros.org/wiki/xacro">
-  <xacro:macro name="arm_ros2_control" params="name hardware_type can_interface baudrate encoder_bw reduction_ratio node_ids joint_indices position_min position_max sync_period_us read_rate_hz state_poll_rate_hz manual_feedback_timeout_ms feedback_stale_timeout_ms enable_emcy_monitor require_full_arm require_position_limits">
+  <xacro:macro name="arm_ros2_control" params="name hardware_type can_interface baudrate encoder_bw reduction_ratio node_ids joint_indices position_min position_max sync_period_us read_rate_hz state_poll_rate_hz manual_feedback_timeout_ms feedback_stale_timeout_ms enable_emcy_monitor max_command_step_rad max_following_error_rad following_error_cycles require_full_arm require_position_limits">
     <ros2_control name="${name}" type="system">
       <hardware>
@@ -35,4 +35,7 @@
           <param name="feedback_stale_timeout_ms">${feedback_stale_timeout_ms}</param>
           <param name="enable_emcy_monitor">${enable_emcy_monitor}</param>
+          <param name="max_command_step_rad">${max_command_step_rad}</param>
+          <param name="max_following_error_rad">${max_following_error_rad}</param>
+          <param name="following_error_cycles">${following_error_cycles}</param>
           <param name="require_full_arm">${require_full_arm}</param>
           <param name="require_position_limits">${require_position_limits}</param>

Commit message: Split remote MoveIt control and stop on disconnect

File: ros2_ws/src/arm_motion_stack/arm_description/urdf/arm.urdf.xacro (robot description, xacro)
@@ -19,4 +19,8 @@
   <xacro:arg name="max_following_error_rad" default="0.05"/>
   <xacro:arg name="following_error_cycles" default="3"/>
+  <xacro:arg name="remote_heartbeat_topic" default="/arm_remote_control/heartbeat"/>
+  <xacro:arg name="remote_profile_fingerprint" default="disabled"/>
+  <xacro:arg name="remote_watchdog_timeout_ms" default="0"/>
+  <xacro:arg name="remote_stop_velocity_threshold_rad_s" default="0.02"/>
   <xacro:arg name="require_full_arm" default="false"/>
   <xacro:arg name="require_position_limits" default="false"/>
@@ -52,4 +56,8 @@
     max_following_error_rad="$(arg max_following_error_rad)"
     following_error_cycles="$(arg following_error_cycles)"
+    remote_heartbeat_topic="$(arg remote_heartbeat_topic)"
+    remote_profile_fingerprint="$(arg remote_profile_fingerprint)"
+    remote_watchdog_timeout_ms="$(arg remote_watchdog_timeout_ms)"
+    remote_stop_velocity_threshold_rad_s="$(arg remote_stop_velocity_threshold_rad_s)"
     require_full_arm="$(arg require_full_arm)"
     require_position_limits="$(arg require_position_limits)"/>

File: ros2_ws/src/arm_motion_stack/arm_description/urdf/ros2_control.xacro (robot description, xacro)
@@ -1,5 +1,5 @@
 <?xml version="1.0"?>
 <robot xmlns:xacro="http://www.ros.org/wiki/xacro">
-  <xacro:macro name="arm_ros2_control" params="name hardware_type can_interface baudrate encoder_bw reduction_ratio node_ids joint_indices position_min position_max sync_period_us read_rate_hz state_poll_rate_hz manual_feedback_timeout_ms feedback_stale_timeout_ms enable_emcy_monitor max_command_step_rad max_following_error_rad following_error_cycles require_full_arm require_position_limits">
+  <xacro:macro name="arm_ros2_control" params="name hardware_type can_interface baudrate encoder_bw reduction_ratio node_ids joint_indices position_min position_max sync_period_us read_rate_hz state_poll_rate_hz manual_feedback_timeout_ms feedback_stale_timeout_ms enable_emcy_monitor max_command_step_rad max_following_error_rad following_error_cycles remote_heartbeat_topic remote_profile_fingerprint remote_watchdog_timeout_ms remote_stop_velocity_threshold_rad_s require_full_arm require_position_limits">
     <ros2_control name="${name}" type="system">
       <hardware>
@@ -38,4 +38,8 @@
           <param name="max_following_error_rad">${max_following_error_rad}</param>
           <param name="following_error_cycles">${following_error_cycles}</param>
+          <param name="remote_heartbeat_topic">${remote_heartbeat_topic}</param>
+          <param name="remote_profile_fingerprint">${remote_profile_fingerprint}</param>
+          <param name="remote_watchdog_timeout_ms">${remote_watchdog_timeout_ms}</param>
+          <param name="remote_stop_velocity_threshold_rad_s">${remote_stop_velocity_threshold_rad_s}</param>
           <param name="require_full_arm">${require_full_arm}</param>
           <param name="require_position_limits">${require_position_limits}</param>
